File: kicad/spinali_mcxn_t1_f9p/gnss.kicad_sch (KiCad schematic)
At the start: 63 parts, among them J3 UART, SW1 SW_SPST, SW2 SW_SPST, U2 PCMF1USB3SZ, U3 AP2112K-3.3, U4 AP2112K-3.3, U5 NEO-F9P-15B

Commit message: fix libraries
Parts:
- BAT1: footprint spinali-connector:JST_SH_SM02B-SRSS-TB_1x02-1MP_P1.00mm_RA -> Connectors:JST_SH_SM02B-SRSS-TB_1x02-1MP_P1.00mm_RA
- SW1, SW2: footprint spinali-connector:Panasonic_EVQPUL_EVQPUC -> Button_Switch_SMD:Panasonic_EVQPUL_EVQPUC
Changed lines of the file:
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@@
 			)
 		)
-		(property "Footprint" "spinali-connector:JST_SH_SM02B-SRSS-TB_1x02-1MP_P1.00mm_RA"
+		(property "Footprint" "Connectors:JST_SH_SM02B-SRSS-TB_1x02-1MP_P1.00mm_RA"
 			(at 119.38 84.836 90)
 			(effects
@@
 			)
 		)
-		(property "Footprint" "spinali-connector:Panasonic_EVQPUL_EVQPUC"
+		(property "Footprint" "Button_Switch_SMD:Panasonic_EVQPUL_EVQPUC"
 			(at 340.36 173.99 0)
 			(effects
@@
 			)
 		)
-		(property "Footprint" "spinali-connector:Panasonic_EVQPUL_EVQPUC"
+		(property "Footprint" "Button_Switch_SMD:Panasonic_EVQPUL_EVQPUC"
 			(at 388.62 173.99 0)
 			(effects
