File: kicad/spinali_mcxn_t1_f9p/gnss.kicad_sch (KiCad schematic)
At the start: 63 parts, among them J3 UART, SW1 SW_SPST, SW2 SW_SPST, U2 PCMF1USB3SZ, U3 AP2112K-3.3, U4 AP2112K-3.3, U5 NEO-F9P-15B

Commit message: Rev A production ready: schematic, layout and BOM fixes
- Rev A production ready.
- Update Resistor R10 on PCB
- Review DNP and re-add I2C pullups (no longer DNP)
- add silkscreen for revision
- Revision in title block
- add revision table
- add silkscreen for battery polarity.
- Changed 0R pull-up / pull-down resistors where possible to 10k for current protection.
- Fixed R13 footprint to correct package -> 0603 (was 0402).
- Improved BOM headers.
- Added Project text variables so Revision, Title, Designers, etc. is set automatically at multiple places.
- Updated all footprints so they match the library again (previously gave DRC error). Now 3D models also work again.
- Moved Time Pulse LED in layout to make it more visible.
- DRC succesfull.
- Added production folder in .gitignore.

Signed-off-by: Youri Tils <youri.tils@nxp.com>
Parts:
- R13: footprint Resistor_SMD:R_0402_1005Metric -> Resistor_SMD:R_0603_1608Metric
- R17, R18: value 0R -> 10k; DigiKey 311-0.0JRCT-ND -> 311-10.0KLRCT-ND; JLCPCB C60485 -> (none); MFPN RC0402JR-070RL -> RC0402FR-0710KL
- R19: value 100K -> 100k
- R20: value 0R SAFEBOOT_N -> 10k; DigiKey 311-0.0JRCT-ND -> 311-10.0KLRCT-ND; MFPN RC0402JR-070RL -> RC0402FR-0710KL
- R29: value 0R RESET_N -> 0R
- R30: value 0R EXTINT -> 0R
- R33: value 0R SPI -> 10k; DigiKey 311-0.0JRCT-ND -> 311-10.0KLRCT-ND; MFPN RC0402JR-070RL -> RC0402FR-0710KL
- R34, R39: value 10K -> 10k
Other:
- note added: "EXTINT"
- note added: "RESET_N"
- note added: "SAFEBOOT_N"
- note added: "SPI"
- company: NXP SEMICONDUCTORS B.V. -> ${COMPANY}
- title: MR-MCXN-T1-F9P -> ${TITLE}
Changed lines of the file:
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@@
 	(paper "A3")
 	(title_block
-		(title "MR-MCXN-T1-F9P")
-		(date "2025-08-27")
-		(rev "X0")
-		(company "NXP SEMICONDUCTORS B.V.")
-		(comment 3 "DESIGNER: YOURI TILS, Iain Galloway")
-		(comment 4 "CTO SYSTEM INNOVATIONS / MOBILE ROBOTICS DOMAIN")
+		(title "${TITLE}")
+		(date "2026-08-21")
+		(rev "${BOARD_REV}")
+		(company "${COMPANY}")
+		(comment 1 "DESIGNER: ${DESIGNER}")
+		(comment 2 "${DEPARTMENT}")
+		(comment 3 "REVIEWED BY: ${REVIEWER}")
 	)
 	(rectangle
@@
 		)
 	)
+	(text "SPI"
+		(exclude_from_sim no)
+		(at 256.794 108.204 0)
+		(effects
+			(font
+				(size 1.27 1.27)
+			)
+		)
+	)
+	(text "SAFEBOOT_N"
+		(exclude_from_sim no)
+		(at 230.886 123.19 0)
+		(effects
+			(font
+				(size 1.27 1.27)
+			)
+		)
+	)
 	(text "NB I_BCKP is only 45uA"
 		(exclude_from_sim no)
@@
 		)
 	)
+	(text "RESET_N"
+		(exclude_from_sim no)
+		(at 238.506 43.434 0)
+		(effects
+			(font
+				(size 1.27 1.27)
+			)
+		)
+	)
 	(text "User Switches\n"
 		(exclude_from_sim no)
@@
 		)
 	)
+	(text "EXTINT"
+		(exclude_from_sim no)
+		(at 237.49 52.324 0)
+		(effects
+			(font
+				(size 1.27 1.27)
+			)
+		)
+	)
 	(text "Need to connect to header\n"
 		(exclude_from_sim no)
@@
 	)
 	(label "+3V3"
-		(at 373.38 161.29 0)
+		(at 368.3 161.29 0)
 		(effects
 			(font
@@
 	)
 	(label "+3V3"
-		(at 325.12 161.29 0)
+		(at 320.04 161.29 0)
 		(effects
 			(font
@@
 		)
 		(instances
-			(project ""
+			(project "spinali_mcxn_t1_f9p"
 				(path "/04285d74-eeba-483c-9378-52bd287e15a2/984519f8-3ba1-4ad2-a1fd-5bc7d7d39895"
 					(reference "C7")
@@
 			)
 		)
-		(property "Value" "100K"
+		(property "Value" "100k"
 			(at 160.02 119.3799 0)
 			(effects
@@
 			)
 		)
-		(property "Value" "0R"
+		(property "Value" "10k"
 			(at 154.94 87.6299 0)
 			(effects
@@
 			)
 		)
-		(property "DigiKey" "311-0.0JRCT-ND"
+		(property "DigiKey" "311-10.0KLRCT-ND"
 			(at 152.4 86.36 0)
 			(effects
@@
 			)
 		)
-		(property "JLCPCB" "C60485"
+		(property "JLCPCB" ""
 			(at 152.4 86.36 0)
 			(effects
@@
 			)
 		)
-		(property "MFPN" "RC0402JR-070RL"
+		(property "MFPN" "RC0402FR-0710KL"
 			(at 152.4 86.36 0)
 			(effects
@@
 		)
 		(instances
-			(project ""
+			(project "spinali_mcxn_t1_f9p"
 				(path "/04285d74-eeba-483c-9378-52bd287e15a2/984519f8-3ba1-4ad2-a1fd-5bc7d7d39895"
 					(reference "ANT1")
@@
 			)
 		)
-		(property "Value" "0R"
+		(property "Value" "10k"
 			(at 154.94 97.7899 0)
 			(effects
@@
 			)
 		)
-		(property "DigiKey" "311-0.0JRCT-ND"
+		(property "DigiKey" "311-10.0KLRCT-ND"
 			(at 152.4 96.52 0)
 			(effects
@@
 			)
 		)
-		(property "JLCPCB" "C60485"
+		(property "JLCPCB" ""
 			(at 152.4 96.52 0)
 			(effects
@@
 			)
 		)
-		(property "MFPN" "RC0402JR-070RL"
+		(property "MFPN" "RC0402FR-0710KL"
 			(at 152.4 96.52 0)
 			(effects
@@
 			)
 		)
-		(property "Value" "0R SPI"
+		(property "Value" "10k"
 			(at 252.73 107.95 90)
 			(effects
@@
 			)
 		)
-		(property "DigiKey" "311-0.0JRCT-ND"
+		(property "DigiKey" "311-10.0KLRCT-ND"
 			(at 252.73 111.76 90)
 			(effects
@@
 			)
 		)
-		(property "MFPN" "RC0402JR-070RL"
+		(property "MFPN" "RC0402FR-0710KL"
 			(at 252.73 111.76 90)
 			(effects
@@
 		)
 		(instances
-			(project ""
+			(project "spinali_mcxn_t1_f9p"
 				(path "/04285d74-eeba-483c-9378-52bd287e15a2/984519f8-3ba1-4ad2-a1fd-5bc7d7d39895"
 					(reference "R33")
@@
 			)
 		)
-		(property "Value" "10K"
+		(property "Value" "10k"
 			(at 378.46 168.9099 0)
 			(effects
@@
 		)
 		(instances
-			(project ""
+			(project "spinali_mcxn_t1_f9p"
 				(path "/04285d74-eeba-483c-9378-52bd287e15a2/984519f8-3ba1-4ad2-a1fd-5bc7d7d39895"
 					(reference "J3")
@@
 			)
 		)
-		(property "Value" "0R RESET_N"
+		(property "Value" "0R"
 			(at 231.14 43.18 90)
 			(effects
@@
 		)
 		(instances
-			(project ""
+			(project "spinali_mcxn_t1_f9p"
 				(path "/04285d74-eeba-483c-9378-52bd287e15a2/984519f8-3ba1-4ad2-a1fd-5bc7d7d39895"
 					(reference "L2")
@@
 			)
 		)
-		(property "Value" "0R EXTINT"
+		(property "Value" "0R"
 			(at 231.14 52.07 90)
 			(effects
@@
 		)
 		(instances
-			(project ""
+			(project "spinali_mcxn_t1_f9p"
 				(path "/04285d74-eeba-483c-9378-52bd287e15a2/984519f8-3ba1-4ad2-a1fd-5bc7d7d39895"
 					(reference "BAT1")
@@
 			)
 		)
-		(property "Footprint" "Resistor_SMD:R_0402_1005Metric"
+		(property "Footprint" "Resistor_SMD:R_0603_1608Metric"
 			(at 74.93 110.998 90)
 			(effects
@@
 		)
 		(instances
-			(project ""
+			(project "spinali_mcxn_t1_f9p"
 				(path "/04285d74-eeba-483c-9378-52bd287e15a2/984519f8-3ba1-4ad2-a1fd-5bc7d7d39895"
 					(reference "R13")
@@
 		)
 		(instances
-			(project ""
+			(project "spinali_mcxn_t1_f9p"
 				(path "/04285d74-eeba-483c-9378-52bd287e15a2/984519f8-3ba1-4ad2-a1fd-5bc7d7d39895"
 					(reference "R21")
@@
 		)
 		(instances
-			(project ""
+			(project "spinali_mcxn_t1_f9p"
 				(path "/04285d74-eeba-483c-9378-52bd287e15a2/984519f8-3ba1-4ad2-a1fd-5bc7d7d39895"
 					(reference "D7")
@@
 		)
 		(instances
-			(project ""
+			(project "spinali_mcxn_t1_f9p"
 				(path "/04285d74-eeba-483c-9378-52bd287e15a2/984519f8-3ba1-4ad2-a1fd-5bc7d7d39895"
 					(reference "D2")
@@
 			)
 		)
-		(property "Value" "0R SAFEBOOT_N"
+		(property "Value" "10k"
 			(at 224.79 120.6499 0)
 			(effects
@@
 			)
 		)
-		(property "DigiKey" "311-0.0JRCT-ND"
+		(property "DigiKey" "311-10.0KLRCT-ND"
 			(at 222.25 119.38 0)
 			(effects
@@
 			)
 		)
-		(property "MFPN" "RC0402JR-070RL"
+		(property "MFPN" "RC0402FR-0710KL"
 			(at 222.25 119.38 0)
 			(effects
@@
 		)
 		(instances
-			(project ""
+			(project "spinali_mcxn_t1_f9p"
 				(path "/04285d74-eeba-483c-9378-52bd287e15a2/984519f8-3ba1-4ad2-a1fd-5bc7d7d39895"
 					(reference "R20")
@@
 		)
 		(instances
-			(project ""
+			(project "spinali_mcxn_t1_f9p"
 				(path "/04285d74-eeba-483c-9378-52bd287e15a2/984519f8-3ba1-4ad2-a1fd-5bc7d7d39895"
 					(reference "D3")
@@
 		)
 		(instances
-			(project ""
+			(project "spinali_mcxn_t1_f9p"
 				(path "/04285d74-eeba-483c-9378-52bd287e15a2/984519f8-3ba1-4ad2-a1fd-5bc7d7d39895"
 					(reference "R41")
@@
 			)
 		)
-		(property "Value" "10K"
+		(property "Value" "10k"
 			(at 330.2 168.9099 0)
 			(effects
