File: kicad/spinali_mcxn_t1_f9p/board-to-board.kicad_sch (KiCad schematic)
At the start: 6 parts, among them J1 DF40TC(4.0)-50DS-0.4V(51), J2 DF40TC(4.0)-50DS-0.4V(51)

Commit message: Rev A production ready: schematic, layout and BOM fixes
- Rev A production ready.
- Update Resistor R10 on PCB
- Review DNP and re-add I2C pullups (no longer DNP)
- add silkscreen for revision
- Revision in title block
- add revision table
- add silkscreen for battery polarity.
- Changed 0R pull-up / pull-down resistors where possible to 10k for current protection.
- Fixed R13 footprint to correct package -> 0603 (was 0402).
- Improved BOM headers.
- Added Project text variables so Revision, Title, Designers, etc. is set automatically at multiple places.
- Updated all footprints so they match the library again (previously gave DRC error). Now 3D models also work again.
- Moved Time Pulse LED in layout to make it more visible.
- DRC succesfull.
- Added production folder in .gitignore.

Signed-off-by: Youri Tils <youri.tils@nxp.com>
Other:
- company: NXP SEMICONDUCTORS B.V. -> ${COMPANY}
- title: MR-MCXN-T1-F9P -> ${TITLE}
