File: kicad/spinali_mcxn_t1_f9p/F9P_Block_Diagram.kicad_sch (KiCad schematic)
At the start: 0 parts

Commit message: Updated block diagrams of F9P, IO and OFLO boards
Signed-off-by: Youri Tils <youri.tils@nxp.com>
Other:
- note added: "3V3"
- note added: "Board-To-Board Connector 1"
- note added: "Board-To-Board Connector 2"
- note added: "DF40TC"
- note added: "EXTINT"
- note added: "FLEXCOMM0_UART"
- note added: "FLEXCOMM3_UART"
- note added: "FLEXCOMM7_UART"
- note added: "FLEXCOMM9_I2C"
- note added: "GPIO 4x FLEXCOMM FLEXIO SmartDMA SDHC0 ADC COMPARATOR FLEXPWM SAI PDM"
- note added: "High Sensitivity Magnetometer RM3100"
- note added: "I3C1"
- note added: "Low-noise LDO"
- note added: "MR-MCXN-T1-Hub"
- note added: "P1_2"
- note added: "P1_22"
- note added: "P1_3"
- note added: "P3_0"
- note added: "P3_7"
- note added: "P3_8"
- note added: "RESET_N"
- note added: "RM3100 sensor suite: PNI 13104: SEN-XY magnetic sensor PNI 13101: SEN-Z magnetic sensor PNI 13156: interface device"
- note added: "UART Connector"
- note added: "USBC"
- note added: "User SW1"
- note added: "User SW2"
- note added: "VBAT RTC 5.0V 1A 3.3V 500mA 1.8V 200mA I3C1 GPIO 3x FLEXCOMM FLEXIO SmartDMA ADC COMPARATOR OPAMP DAC FLEXPWM"
- note removed: "GPIO SDHC0 SmartDMA FLEXCOMM0 FLEXCOMM3 FLEXCOMM7 FLEXIO"
- note removed: "GPXFIX"
- note removed: "High Sensitivity Magnetometer RM3100 sensor suite: PNI 13104: SEN-XY magnetic sensor PNI 13101: SEN-Z magnetic sensor PNI 13156: interface device"
- note removed: "I2C_4"
- note removed: "I2C_9 (optional)"
- note removed: "J1"
- note removed: "J2"
- note removed: "J8"
- note removed: "J9"
- note removed: "LDO"
- note removed: "MR-MCXN-T1 Hub Connectors"
- note removed: "MR-MCXN-T1-F9P Shield Connectors"
- note removed: "UART (external RTK corrections input)"
- note removed: "UART0"
- note removed: "UART3"
- note removed: "UART7"
- note removed: "USB (Configuration)"
- note removed: "Vbatt 5.0V 3.3V 1.8V I3C (I2C) GPIO FLEXCOMM2 FLEXCOMM4 FLEXCOMM6 FLEXIO_0 Analog OPAMP DAC"
- note removed: "Vbatt 5.0V 3.3V 1.8V I3C (I2C_4) GPIO FLEXCOMM2 FLEXCOMM4 FLEXCOMM6 FLEXIO_0 Analog OPAMP DAC"
