File: kicad/spinali_mcxn_t1_oflo/board-to-board.kicad_sch (KiCad schematic)
At the start: 6 parts, among them J1 DF40TC(4.0)-50DS-0.4V(51), J2 DF40TC(4.0)-50DS-0.4V(51)

Commit message: Finish rename and org.
Signed-off-by: Benjamin Perseghetti <bperseghetti@rudislabs.com>
Other:
- title: MR-MCXN-T1 Optical Flow -> MR-MCXN-T1-OFLO
