File: kicad/spinali_mcxn_t1_oflo/board-to-board.kicad_sch (KiCad schematic)
At the start: 6 parts, among them J1 DF40TC(4.0)-50DS-0.4V(51), J2 DF40TC(4.0)-50DS-0.4V(51)

Commit message: Added Rev-A in MR-MCXN-T1-OFLO
- Added Rev-A in schematic and layout
- Created production files

Signed-off-by: Youri Tils <youri.tils@nxp.com>
Other:
- company: NXP SEMICONDUCTORS B.V. -> ${COMPANY}
- title: MR-MCXN-T1-OFLO -> ${TITLE}
Changed lines of the file:
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@@
 	(paper "A4")
 	(title_block
-		(title "MR-MCXN-T1-OFLO")
-		(date "2025-04-16")
-		(rev "X0")
-		(company "NXP SEMICONDUCTORS B.V.")
-		(comment 3 "DESIGNER: YOURI TILS")
-		(comment 4 "CTO SYSTEM INNOVATIONS / MOBILE ROBOTICS DOMAIN")
+		(title "${TITLE}")
+		(date "2026-08-24")
+		(rev "${BOARD_REV}")
+		(company "${COMPANY}")
+		(comment 1 "DESIGNER: ${DESIGNER}")
+		(comment 2 "${DEPARTMENT}")
+		(comment 3 "REVIEWED BY: ${REVIEWER}")
 	)
 	(text "300mA max per pin\n5V = 1A max\n3V3 = 500mA max\n1V8 = 200mA max"
@@
 		)
 		(instances
-			(project ""
+			(project "spinali_mcxn_t1_oflo"
 				(path "/04285d74-eeba-483c-9378-52bd287e15a2/ccc0d483-c16f-4a48-802e-c15323fec247"
 					(reference "J1")
