File: kicad/spinali_mcxn_t1_oflo/sensors.kicad_sch (KiCad schematic)
At the start: 42 parts, among them Q1 BC817, Q2 BC868, Q3 BC807, U1 AFBR-S50LX85D, U2 PAA3905E1, U3 ICM-45686, U4 ICM-42688-P

Commit message: Finish rename and org.
Signed-off-by: Benjamin Perseghetti <bperseghetti@rudislabs.com>
Other:
- title: MR-MCXN-T1 Optical Flow -> MR-MCXN-T1-OFLO
