File: kicad/spinali_mcxn_t1_oflo/sensors.kicad_sch (KiCad schematic)
At the start: 42 parts, among them Q1 BC817, Q2 BC868, Q3 BC807, U1 AFBR-S50LX85D, U2 PAA3905E1, U3 ICM-45686, U4 ICM-42688-P

Commit message: Added Rev-A in MR-MCXN-T1-OFLO
- Added Rev-A in schematic and layout
- Created production files

Signed-off-by: Youri Tils <youri.tils@nxp.com>
Other:
- company: NXP SEMICONDUCTORS B.V. -> ${COMPANY}
- title: MR-MCXN-T1-OFLO -> ${TITLE}
Changed lines of the file:
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@@
 	(paper "A4")
 	(title_block
-		(title "MR-MCXN-T1-OFLO")
-		(date "2025-04-16")
-		(rev "X0")
-		(company "NXP SEMICONDUCTORS B.V.")
-		(comment 3 "DESIGNER: YOURI TILS")
-		(comment 4 "CTO SYSTEM INNOVATIONS / MOBILE ROBOTICS DOMAIN")
+		(title "${TITLE}")
+		(date "2026-08-24")
+		(rev "${BOARD_REV}")
+		(company "${COMPANY}")
+		(comment 1 "DESIGNER: ${DESIGNER}")
+		(comment 2 "${DEPARTMENT}")
+		(comment 3 "REVIEWED BY: ${REVIEWER}")
 	)
 	(text "325mA"
@@
 		)
 		(instances
-			(project ""
+			(project "spinali_mcxn_t1_oflo"
 				(path "/04285d74-eeba-483c-9378-52bd287e15a2/d46d18ea-5041-4bdf-8a2f-871da180f13d"
 					(reference "U1")
@@
 		)
 		(instances
-			(project ""
+			(project "spinali_mcxn_t1_oflo"
 				(path "/04285d74-eeba-483c-9378-52bd287e15a2/d46d18ea-5041-4bdf-8a2f-871da180f13d"
 					(reference "C3")
@@
 		)
 		(instances
-			(project ""
+			(project "spinali_mcxn_t1_oflo"
 				(path "/04285d74-eeba-483c-9378-52bd287e15a2/d46d18ea-5041-4bdf-8a2f-871da180f13d"
 					(reference "R1")
@@
 		)
 		(instances
-			(project ""
+			(project "spinali_mcxn_t1_oflo"
 				(path "/04285d74-eeba-483c-9378-52bd287e15a2/d46d18ea-5041-4bdf-8a2f-871da180f13d"
 					(reference "U2")
@@
 		)
 		(instances
-			(project ""
+			(project "spinali_mcxn_t1_oflo"
 				(path "/04285d74-eeba-483c-9378-52bd287e15a2/d46d18ea-5041-4bdf-8a2f-871da180f13d"
 					(reference "D1")
@@
 		)
 		(instances
-			(project ""
+			(project "spinali_mcxn_t1_oflo"
 				(path "/04285d74-eeba-483c-9378-52bd287e15a2/d46d18ea-5041-4bdf-8a2f-871da180f13d"
 					(reference "R2")
@@
 		)
 		(instances
-			(project ""
+			(project "spinali_mcxn_t1_oflo"
 				(path "/04285d74-eeba-483c-9378-52bd287e15a2/d46d18ea-5041-4bdf-8a2f-871da180f13d"
 					(reference "R3")
@@
 		)
 		(instances
-			(project ""
+			(project "spinali_mcxn_t1_oflo"
 				(path "/04285d74-eeba-483c-9378-52bd287e15a2/d46d18ea-5041-4bdf-8a2f-871da180f13d"
 					(reference "Q1")
@@
 		)
 		(instances
-			(project ""
+			(project "spinali_mcxn_t1_oflo"
 				(path "/04285d74-eeba-483c-9378-52bd287e15a2/d46d18ea-5041-4bdf-8a2f-871da180f13d"
 					(reference "U4")
@@
 		)
 		(instances
-			(project ""
+			(project "spinali_mcxn_t1_oflo"
 				(path "/04285d74-eeba-483c-9378-52bd287e15a2/d46d18ea-5041-4bdf-8a2f-871da180f13d"
 					(reference "R6")
@@
 		)
 		(instances
-			(project ""
+			(project "spinali_mcxn_t1_oflo"
 				(path "/04285d74-eeba-483c-9378-52bd287e15a2/d46d18ea-5041-4bdf-8a2f-871da180f13d"
 					(reference "TP3")
@@
 		)
 		(instances
-			(project ""
+			(project "spinali_mcxn_t1_oflo"
 				(path "/04285d74-eeba-483c-9378-52bd287e15a2/d46d18ea-5041-4bdf-8a2f-871da180f13d"
 					(reference "L1")
@@
 		)
 		(instances
-			(project ""
+			(project "spinali_mcxn_t1_oflo"
 				(path "/04285d74-eeba-483c-9378-52bd287e15a2/d46d18ea-5041-4bdf-8a2f-871da180f13d"
 					(reference "U3")
@@
 		)
 		(instances
-			(project ""
+			(project "spinali_mcxn_t1_oflo"
 				(path "/04285d74-eeba-483c-9378-52bd287e15a2/d46d18ea-5041-4bdf-8a2f-871da180f13d"
 					(reference "TP1")
@@
 		)
 		(instances
-			(project ""
+			(project "spinali_mcxn_t1_oflo"
 				(path "/04285d74-eeba-483c-9378-52bd287e15a2/d46d18ea-5041-4bdf-8a2f-871da180f13d"
 					(reference "Q3")
