File: kicad/spinali_mcxn_t1_oflo/spinali_mcxn_t1_oflo.kicad_pcb (KiCad board)
At the start: 4 copper layers, 36.5 x 46 mm, 49 parts, among them J1 DF40TC(4.0)-50DS-0.4V(51), J2 DF40TC(4.0)-50DS-0.4V(51), Q1 BC817, Q2 BC868, Q3 BC807, U1 AFBR-S50LX85D, U2 PAA3905E1, U3 ICM-45686, U4 ICM-42688-P

Commit message: Added Rev-A in MR-MCXN-T1-OFLO
- Added Rev-A in schematic and layout
- Created production files

Signed-off-by: Youri Tils <youri.tils@nxp.com>
Other:
- board text added: "Rev ${BOARD_REV}"
