File: kicad/spinali_mcxn_t1_io/spinali_mcxn_t1_io.kicad_pcb (KiCad board)
At the start: 4 copper layers, 36.5 x 46 mm, 85 parts, among them J1 DF40TC(4.0)-50DS-0.4V(51), J10 SPI2, J11 ESC1, J12 ESC2, J13 RTC_BAT, J2 DF40TC(4.0)-50DS-0.4V(51), J3 I2C1, J4 I2C2, J5 UART1, J6 UART2, J7 QDEC, J8 GPS, J9 SPI1, Q1 NX138BKMYL, SW1 CHS-01TA

Commit message: Updated MR-MCXN-T1 IO board for production version X1
- Changed R10 and R11 to 10k and DNP, so they work with the latest MR-MCXN-T1 hub version X1
- Updated page information to version X1

Signed-off-by: Youri Tils <youri.tils@nxp.com>
Parts:
- J3: value I2C1 -> I3C
- J4: value I2C2 -> I2C
- R10, R11: value 4k7 -> 10k
Changed lines of the file:
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@@
 			)
 		)
-		(property "Value" "4k7"
+		(property "Value" "10k"
 			(at 0 1.43 90)
 			(layer "F.Fab")
@@
 			)
 		)
-		(property "DigiKey" "311-4.70KHRCT-ND"
+		(property "DigiKey" "311-10.0KHRCT-ND"
 			(at 0 0 270)
 			(unlocked yes)
@@
 			)
 		)
-		(property "MFPN" "RC0603FR-074K7L"
+		(property "MFPN" "RC0603FR-0710KL"
 			(at 0 0 270)
 			(unlocked yes)
@@
 		(sheetname "/Board-to-Board/")
 		(sheetfile "board-to-board.kicad_sch")
-		(attr smd)
+		(attr smd dnp)
 		(fp_line
 			(start -0.237258 0.5225)
@@
 		(model "${KICAD9_3DMODEL_DIR}/Connector_JST.3dshapes/JST_SH_SM08B-SRSS-TB_1x08-1MP_P1.00mm_Horizontal.step"
 			(offset
-				(xyz 0 -2.5 1.5)
+				(xyz 0 0 0)
 			)
 			(scale
@@
 			)
 			(rotate
-				(xyz -90 -0 -0)
+				(xyz -0 -0 -0)
 			)
 		)
@@
 		)
 		(property "Value" "RTC_BAT"
-			(at -3.3 -0.2 180)
+			(at -3.3 -0.2 0)
 			(layer "F.SilkS")
 			(effects
@@
 			)
 			(rotate
-				(xyz -90 -0 -0)
+				(xyz -0 -0 -0)
 			)
 		)
@@
 			)
 		)
-		(property "Value" "I2C2"
+		(property "Value" "I2C"
 			(at -5.4125 -0.2 90)
 			(layer "F.SilkS")
@@
 		(tags "connector JST SH horizontal")
 		(property "Reference" "J12"
-			(at 6.35 -0.6 180)
+			(at 6.35 -0.6 0)
 			(layer "F.SilkS")
 			(hide yes)
@@
 		)
 		(property "Value" "ESC2"
-			(at 6.3 -1.4 180)
+			(at 6.3 -1.4 0)
 			(layer "F.SilkS")
 			(effects
@@
 		(model "${KICAD9_3DMODEL_DIR}/Connector_JST.3dshapes/JST_SH_SM08B-SRSS-TB_1x08-1MP_P1.00mm_Horizontal.step"
 			(offset
-				(xyz 0 -2.5 1.5)
+				(xyz 0 0 0)
 			)
 			(scale
@@
 			)
 			(rotate
-				(xyz -90 -0 -0)
+				(xyz -0 -0 -0)
 			)
 		)
@@
 			)
 		)
-		(property "Value" "I2C1"
+		(property "Value" "I3C"
 			(at 5.325 -0.25 90)
 			(layer "F.SilkS")
@@
 			)
 		)
-		(property "Value" "4k7"
+		(property "Value" "10k"
 			(at 0 1.43 90)
 			(layer "F.Fab")
@@
 			)
 		)
-		(property "DigiKey" "311-4.70KHRCT-ND"
+		(property "DigiKey" "311-10.0KHRCT-ND"
 			(at 0 0 270)
 			(unlocked yes)
@@
 			)
 		)
-		(property "MFPN" "RC0603FR-074K7L"
+		(property "MFPN" "RC0603FR-0710KL"
 			(at 0 0 270)
 			(unlocked yes)
@@
 		(sheetname "/Board-to-Board/")
 		(sheetfile "board-to-board.kicad_sch")
-		(attr smd)
+		(attr smd dnp)
 		(fp_line
 			(start -0.237258 0.5225)
