File: kicad/spinali_mcxn_t1_io/spinali_mcxn_t1_io.kicad_pcb (KiCad board)
At the start: 4 copper layers, 36.5 x 46 mm, 85 parts, among them J1 DF40TC(4.0)-50DS-0.4V(51), J10 SPI2, J11 ESC1, J12 ESC2, J13 RTC_BAT, J2 DF40TC(4.0)-50DS-0.4V(51), J3 I3C, J4 I2C, J5 UART1, J6 UART2, J7 QDEC, J8 GPS, J9 SPI1, Q1 NX138BKMYL, SW1 CHS-01TA

Commit message: Added Rev-A in MR-MCXN-T1-IO
- Added Rev-A in schematic and layout
- Created production files

Signed-off-by: Youri Tils <youri.tils@nxp.com>
Other:
- board text added: "Rev ${BOARD_REV}"
