File: kicad/spinali_mcxn_t1_io/board-to-board.kicad_sch (KiCad schematic)
At the start: 10 parts, among them J1 DF40TC(4.0)-50DS-0.4V(51), J2 DF40TC(4.0)-50DS-0.4V(51)

Commit message: Updated MR-MCXN-T1 IO board for production version X1
- Changed R10 and R11 to 10k and DNP, so they work with the latest MR-MCXN-T1 hub version X1
- Updated page information to version X1

Signed-off-by: Youri Tils <youri.tils@nxp.com>
Parts:
- R10, R11: value 4k7 -> 10k; DigiKey 311-4.70KHRCT-ND -> 311-10.0KHRCT-ND; MFPN RC0603FR-074K7L -> RC0603FR-0710KL; now not fitted
Changed lines of the file:
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@@
 	(title_block
 		(title "MR-MCXN-T1-IO")
-		(date "2025-10-13")
-		(rev "X0")
+		(date "2026-07-24")
+		(rev "X1")
 		(company "NXP SEMICONDUCTORS B.V.")
-		(comment 3 "DESIGNER: YOURI TILS")
-		(comment 4 "CTO SYSTEM INNOVATIONS / MOBILE ROBOTICS DOMAIN")
+		(comment 1 "DESIGNER: YOURI TILS")
+		(comment 2 "CTO SYSTEM INNOVATIONS / MOBILE ROBOTICS DOMAIN")
 	)
 	(text "300mA max per pin\n5V = 1A max\n3V3 = 500mA max\n1V8 = 200mA max"
@@
 		(in_bom yes)
 		(on_board yes)
-		(dnp no)
+		(dnp yes)
 		(fields_autoplaced yes)
 		(property "Reference" "R10"
@@
 			)
 		)
-		(property "Value" "4k7"
+		(property "Value" "10k"
 			(at 53.34 78.7399 0)
 			(effects
@@
 			)
 		)
-		(property "DigiKey" "311-4.70KHRCT-ND"
+		(property "DigiKey" "311-10.0KHRCT-ND"
 			(at 50.8 77.47 0)
 			(effects
@@
 			)
 		)
-		(property "MFPN" "RC0603FR-074K7L"
+		(property "MFPN" "RC0603FR-0710KL"
 			(at 50.8 77.47 0)
 			(effects
@@
 		(in_bom yes)
 		(on_board yes)
-		(dnp no)
+		(dnp yes)
 		(fields_autoplaced yes)
 		(property "Reference" "R11"
@@
 			)
 		)
-		(property "Value" "4k7"
+		(property "Value" "10k"
 			(at 62.23 78.7399 0)
 			(effects
@@
 			)
 		)
-		(property "DigiKey" "311-4.70KHRCT-ND"
+		(property "DigiKey" "311-10.0KHRCT-ND"
 			(at 59.69 77.47 0)
 			(effects
@@
 			)
 		)
-		(property "MFPN" "RC0603FR-074K7L"
+		(property "MFPN" "RC0603FR-0710KL"
 			(at 59.69 77.47 0)
 			(effects

Commit message: Added Rev-A in MR-MCXN-T1-IO
- Added Rev-A in schematic and layout
- Created production files

Signed-off-by: Youri Tils <youri.tils@nxp.com>
Other:
- company: NXP SEMICONDUCTORS B.V. -> ${COMPANY}
- title: MR-MCXN-T1-IO -> ${TITLE}
