File: kicad/spinali_mcxn_t1_io/io1.kicad_sch (KiCad schematic)
At the start: 35 parts, among them J10 SPI2, J3 I2C1, J4 I2C2, J5 UART1, J6 UART2, J7 QDEC, J9 SPI1

Commit message: Updated MR-MCXN-T1 IO board for production version X1
- Changed R10 and R11 to 10k and DNP, so they work with the latest MR-MCXN-T1 hub version X1
- Updated page information to version X1

Signed-off-by: Youri Tils <youri.tils@nxp.com>
Parts:
- J3: value I2C1 -> I3C
- J4: value I2C2 -> I2C
Connections:
- net at D2.5 (IO_4): now also D2.6 (NC_1)
- net at D1.5 (IO_4): now also D1.6 (NC_1)
Changed lines of the file:
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@@
 	(title_block
 		(title "MR-MCXN-T1-IO")
-		(date "2025-10-13")
-		(rev "X0")
+		(date "2026-07-24")
+		(rev "X1")
 		(company "NXP SEMICONDUCTORS B.V.")
-		(comment 3 "DESIGNER: YOURI TILS")
-		(comment 4 "CTO SYSTEM INNOVATIONS / MOBILE ROBOTICS DOMAIN")
+		(comment 1 "DESIGNER: YOURI TILS")
+		(comment 2 "CTO SYSTEM INNOVATIONS / MOBILE ROBOTICS DOMAIN")
 	)
 	(junction
@@
 			)
 		)
-		(property "Value" "I2C2"
+		(property "Value" "I2C"
 			(at 182.88 103.5049 0)
 			(effects
@@
 			)
 		)
-		(property "Value" "I2C1"
+		(property "Value" "I3C"
 			(at 182.88 64.1349 0)
 			(effects

Commit message: Added Rev-A in MR-MCXN-T1-IO
- Added Rev-A in schematic and layout
- Created production files

Signed-off-by: Youri Tils <youri.tils@nxp.com>
Connections:
- net at D2.5 (IO_4): now also D2.6 (NC_1)
- net at D1.5 (IO_4): now also D1.6 (NC_1)
Other:
- company: NXP SEMICONDUCTORS B.V. -> ${COMPANY}
- title: MR-MCXN-T1-IO -> ${TITLE}
Changed lines of the file:
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@@
 	(paper "A3")
 	(title_block
-		(title "MR-MCXN-T1-IO")
-		(date "2026-07-24")
-		(rev "X1")
-		(company "NXP SEMICONDUCTORS B.V.")
-		(comment 1 "DESIGNER: YOURI TILS")
-		(comment 2 "CTO SYSTEM INNOVATIONS / MOBILE ROBOTICS DOMAIN")
+		(title "${TITLE}")
+		(date "2026-08-24")
+		(rev "${BOARD_REV}")
+		(company "${COMPANY}")
+		(comment 1 "DESIGNER: ${DESIGNER}")
+		(comment 2 "${DEPARTMENT}")
+		(comment 3 "REVIEWED BY: ${REVIEWER}")
 	)
 	(junction
@@
 		)
 		(instances
-			(project ""
+			(project "spinali_mcxn_t1_io"
 				(path "/04285d74-eeba-483c-9378-52bd287e15a2/3c5f83e0-e92e-42ae-8f83-967e4a3fe88f"
 					(reference "C1")
@@
 		)
 		(instances
-			(project ""
+			(project "spinali_mcxn_t1_io"
 				(path "/04285d74-eeba-483c-9378-52bd287e15a2/3c5f83e0-e92e-42ae-8f83-967e4a3fe88f"
 					(reference "D4")
@@
 		)
 		(instances
-			(project ""
+			(project "spinali_mcxn_t1_io"
 				(path "/04285d74-eeba-483c-9378-52bd287e15a2/3c5f83e0-e92e-42ae-8f83-967e4a3fe88f"
 					(reference "C2")
