File: kicad/spinali_mcxn_t1_io/io2.kicad_sch (KiCad schematic)
At the start: 39 parts, among them J11 ESC1, J12 ESC2, J13 RTC_BAT, J8 GPS, Q1 NX138BKMYL, SW1 CHS-01TA

Commit message: Added Rev-A in MR-MCXN-T1-IO
- Added Rev-A in schematic and layout
- Created production files

Signed-off-by: Youri Tils <youri.tils@nxp.com>
Other:
- company: NXP SEMICONDUCTORS B.V. -> ${COMPANY}
- title: MR-MCXN-T1-IO -> ${TITLE}
Changed lines of the file:
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@@
 	(paper "A3")
 	(title_block
-		(title "MR-MCXN-T1-IO")
-		(date "2026-07-24")
-		(rev "X1")
-		(company "NXP SEMICONDUCTORS B.V.")
-		(comment 1 "DESIGNER: YOURI TILS")
-		(comment 2 "CTO SYSTEM INNOVATIONS / MOBILE ROBOTICS DOMAIN")
+		(title "${TITLE}")
+		(date "2026-08-24")
+		(rev "${BOARD_REV}")
+		(company "${COMPANY}")
+		(comment 1 "DESIGNER: ${DESIGNER}")
+		(comment 2 "${DEPARTMENT}")
+		(comment 3 "REVIEWED BY: ${REVIEWER}")
 	)
 	(text "1/16 divider"
@@
 		)
 		(instances
-			(project ""
+			(project "spinali_mcxn_t1_io"
 				(path "/04285d74-eeba-483c-9378-52bd287e15a2/9be56f45-5afd-411f-a1bb-7adb647427b1"
 					(reference "SW1")
@@
 		)
 		(instances
-			(project ""
+			(project "spinali_mcxn_t1_io"
 				(path "/04285d74-eeba-483c-9378-52bd287e15a2/9be56f45-5afd-411f-a1bb-7adb647427b1"
 					(reference "C19")
@@
 		)
 		(instances
-			(project ""
+			(project "spinali_mcxn_t1_io"
 				(path "/04285d74-eeba-483c-9378-52bd287e15a2/9be56f45-5afd-411f-a1bb-7adb647427b1"
 					(reference "R16")
@@
 		)
 		(instances
-			(project ""
+			(project "spinali_mcxn_t1_io"
 				(path "/04285d74-eeba-483c-9378-52bd287e15a2/9be56f45-5afd-411f-a1bb-7adb647427b1"
 					(reference "C20")
@@
 		)
 		(instances
-			(project ""
+			(project "spinali_mcxn_t1_io"
 				(path "/04285d74-eeba-483c-9378-52bd287e15a2/9be56f45-5afd-411f-a1bb-7adb647427b1"
 					(reference "D20")
@@
 		)
 		(instances
-			(project ""
+			(project "spinali_mcxn_t1_io"
 				(path "/04285d74-eeba-483c-9378-52bd287e15a2/9be56f45-5afd-411f-a1bb-7adb647427b1"
 					(reference "R3")
@@
 		)
 		(instances
-			(project ""
+			(project "spinali_mcxn_t1_io"
 				(path "/04285d74-eeba-483c-9378-52bd287e15a2/9be56f45-5afd-411f-a1bb-7adb647427b1"
 					(reference "D15")
@@
 		)
 		(instances
-			(project ""
+			(project "spinali_mcxn_t1_io"
 				(path "/04285d74-eeba-483c-9378-52bd287e15a2/9be56f45-5afd-411f-a1bb-7adb647427b1"
 					(reference "R1")
@@
 		)
 		(instances
-			(project ""
+			(project "spinali_mcxn_t1_io"
 				(path "/04285d74-eeba-483c-9378-52bd287e15a2/9be56f45-5afd-411f-a1bb-7adb647427b1"
 					(reference "Q1")
@@
 		)
 		(instances
-			(project ""
+			(project "spinali_mcxn_t1_io"
 				(path "/04285d74-eeba-483c-9378-52bd287e15a2/9be56f45-5afd-411f-a1bb-7adb647427b1"
 					(reference "J13")
